File: hardware/esp12f-si7021/esp12f-si7021.kicad_pcb (KiCad board)
At the start: 2 copper layers, 49.9 x 34 mm, 25 parts, among them J2 UART, Q1 BSS84, Q2 BSS84, U1 MCP1700-3302E_SOT23, U2 ESP-12F, U3 Si7021-A20

Commit message: Add case, analysis
Parts:
- U1: value MCP1700-3302E_SOT23 -> MCP1700
Changed lines of the file:
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@@
   (layers
     (0 F.Cu signal)
-    (31 B.Cu signal)
+    (31 B.Cu signal hide)
     (32 B.Adhes user hide)
     (33 F.Adhes user hide)
     (34 B.Paste user hide)
-    (35 F.Paste user)
+    (35 F.Paste user hide)
     (36 B.SilkS user hide)
-    (37 F.SilkS user)
+    (37 F.SilkS user hide)
     (38 B.Mask user hide)
     (39 F.Mask user hide)
@@
     (42 Eco1.User user hide)
     (43 Eco2.User user hide)
-    (44 Edge.Cuts user hide)
+    (44 Edge.Cuts user)
     (45 Margin user)
-    (46 B.CrtYd user hide)
+    (46 B.CrtYd user)
     (47 F.CrtYd user)
-    (48 B.Fab user hide)
-    (49 F.Fab user)
+    (48 B.Fab user)
+    (49 F.Fab user hide)
   )
   (setup
-    (last_trace_width 0.75)
+    (last_trace_width 0.25)
     (user_trace_width 0.25)
     (user_trace_width 0.5)
@@
     (aux_axis_origin 0 0)
     (grid_origin 0 34)
-    (visible_elements FFFFEF7F)
+    (visible_elements FFFFE77F)
     (pcbplotparams
       (layerselection 0x010f8_ffffffff)
@@
       (effects (font (size 1 1) (thickness 0.15)))
     )
-    (fp_text value UART (at 1.575 2.75) (layer F.Fab)
+    (fp_text value UART (at 3.44744 -0.21444) (layer F.Fab)
       (effects (font (size 1 1) (thickness 0.15)))
     )
@@
       (effects (font (size 1 1) (thickness 0.15)))
     )
-    (fp_text value 1uF (at 0 1.82) (layer F.Fab)
+    (fp_text value 1uF (at 0.19398 2.19964) (layer F.Fab)
       (effects (font (size 1 1) (thickness 0.15)))
     )
@@
       (effects (font (size 1 1) (thickness 0.15)))
     )
-    (fp_text value Download (at 0 1.9) (layer F.Fab)
+    (fp_text value Download (at -0.34544 -2.27076) (layer F.Fab)
       (effects (font (size 1 1) (thickness 0.15)))
     )
@@
       (effects (font (size 1 1) (thickness 0.15)))
     )
-    (fp_text value "JST GH2" (at 0 3.9) (layer F.Fab)
+    (fp_text value "JST GH2" (at 0.2174 1.67004) (layer F.Fab)
       (effects (font (size 1 1) (thickness 0.15)))
     )
@@
       (effects (font (size 1 1) (thickness 0.15)))
     )
-    (fp_text value ESP-12F (at -0.06 -12.78 90) (layer F.Fab)
+    (fp_text value ESP-12F (at 0.274 2.024 90) (layer F.Fab)
       (effects (font (size 1 1) (thickness 0.15)))
     )
@@
       (effects (font (size 1 1) (thickness 0.15)))
     )
-    (fp_text value 10K (at 0 1.82) (layer F.Fab)
+    (fp_text value 10K (at 0 -1.69164) (layer F.Fab)
       (effects (font (size 1 1) (thickness 0.15)))
     )
@@
       (effects (font (size 1 1) (thickness 0.15)))
     )
-    (fp_text value MCP1700-3302E_SOT23 (at 3.66268 -1.6764 90) (layer F.Fab)
+    (fp_text value MCP1700 (at 4.17576 -1.96596 90) (layer F.Fab)
       (effects (font (size 1 1) (thickness 0.15)))
     )
@@
       (effects (font (size 1 1) (thickness 0.15)))
     )
-    (fp_text value 100K (at -0.43594 1.68656 90) (layer F.Fab)
+    (fp_text value 100K (at -0.3953 1.9558 90) (layer F.Fab)
       (effects (font (size 1 1) (thickness 0.15)))
     )
@@
       (effects (font (size 1 1) (thickness 0.15)))
     )
-    (fp_text value 330K (at 0 1.82 90) (layer F.Fab)
+    (fp_text value 330K (at -0.1635 2.032 90) (layer F.Fab)
       (effects (font (size 1 1) (thickness 0.15)))
     )
@@
       (effects (font (size 1 1) (thickness 0.15)))
     )
-    (fp_text value Si7021-A20 (at -3.23088 0.11684 180) (layer F.Fab)
+    (fp_text value Si7021-A20 (at -3.683 2.159 180) (layer F.Fab)
       (effects (font (size 1 1) (thickness 0.15)))
     )
@@
       (effects (font (size 1 1) (thickness 0.15)))
     )
-    (fp_text value 0.1uF (at 0.03462 -2.16916 90) (layer F.Fab)
+    (fp_text value 0.1uF (at -4.7863 0.0254 90) (layer F.Fab)
       (effects (font (size 1 1) (thickness 0.15)))
     )
@@
       (effects (font (size 1 1) (thickness 0.15)))
     )
-    (fp_text value 10uF (at 0 1.82 90) (layer F.Fab)
+    (fp_text value 10uF (at -0.3413 2.1336 90) (layer F.Fab)
       (effects (font (size 1 1) (thickness 0.15)))
     )
@@
       (effects (font (size 1 1) (thickness 0.15)))
     )
-    (fp_text value 0.1uF (at 0 1.82 90) (layer F.Fab)
+    (fp_text value 0.1uF (at 0.0365 -1.778 90) (layer F.Fab)
       (effects (font (size 1 1) (thickness 0.15)))
     )
@@
     (connect_pads (clearance 0.508))
     (min_thickness 0.254)
-    (fill yes (arc_segments 32) (thermal_gap 0.508) (thermal_bridge_width 0.508))
+    (fill (arc_segments 32) (thermal_gap 0.508) (thermal_bridge_width 0.508))
     (polygon
       (pts
@@
     (connect_pads (clearance 0.508))
     (min_thickness 0.254)
-    (fill yes (arc_segments 32) (thermal_gap 0.508) (thermal_bridge_width 0.508))
+    (fill (arc_segments 32) (thermal_gap 0.508) (thermal_bridge_width 0.508))
     (polygon
       (pts
